Commit message: Gaze integration tested. Robot tested successfully. Started new XACRO.

File: src/universal_robot/ur_description/urdf/Sur10.urdf.xacro (robot description, xacro)
@@ -4,7 +4,8 @@
   Author: Kelsey Hawkins
   Contributers: Jimmy Da Silva, Ajit Krisshna N L, Muhammad Asif Rana
+  Nuno Pereira!!!
 -->
-  <xacro:include filename="$(find ur_description)/urdf/ur.transmission.xacro" />
-  <xacro:include filename="$(find ur_description)/urdf/ur.gazebo.xacro" />
+  <!-- <xacro:include filename="$(find ur_description)/urdf/ur.transmission.xacro" />
+  <xacro:include filename="$(find ur_description)/urdf/ur.gazebo.xacro" /> -->
   <xacro:macro name="cylinder_inertial" params="radius length mass *origin">
     <inertial>
@@ -32,5 +33,6 @@
      <!-- forearm_lower_limit:=${-pi}    forearm_upper_limit:=${pi} -->
     <!-- Inertia parameters -->
-    <xacro:property name="base_mass" value="4.0" />  <!-- This mass might be incorrect -->
+    <!-- This mass might be incorrect -->
+    <!-- <xacro:property name="base_mass" value="4.0" />
     <xacro:property name="shoulder_mass" value="7.778" />
     <xacro:property name="upper_arm_mass" value="12.93" />
@@ -38,5 +40,5 @@
     <xacro:property name="wrist_1_mass" value="1.96" />
     <xacro:property name="wrist_2_mass" value="1.96" />
-    <xacro:property name="wrist_3_mass" value="0.202" />
+    <xacro:property name="wrist_3_mass" value="0.202" /> -->
     <!-- These parameters are borrowed from the urcontrol.conf file
         but are not verified for the correct permutation.
@@ -51,20 +53,20 @@
     <!-- Kinematic model -->
     <!-- Properties from urcontrol.conf -->
-    <xacro:property name="d1" value="0.1273" />
+    <!-- <xacro:property name="d1" value="0.1273" />
     <xacro:property name="a2" value="-0.612" />
     <xacro:property name="a3" value="-0.5723" />
     <xacro:property name="d4" value="0.163941" />
     <xacro:property name="d5" value="0.1157" />
-    <xacro:property name="d6" value="0.0922" />
+    <xacro:property name="d6" value="0.0922" /> -->
     <!-- Arbitrary offsets for shoulder/elbow joints -->
-    <xacro:property name="shoulder_offset" value="0.220941" />  <!-- measured from model -->
-    <xacro:property name="elbow_offset" value="-0.1719" /> <!-- measured from model -->
+    <!-- <xacro:property name="shoulder_offset" value="0.220941" />   -->
+    <!-- <xacro:property name="elbow_offset" value="-0.1719" />  -->
     <!-- link lengths used in model -->
-    <xacro:property name="shoulder_height" value="${d1}" />
-    <xacro:property name="upper_arm_length" value="${-a2}" />
-    <xacro:property name="forearm_length" value="${-a3}" />
-    <xacro:property name="wrist_1_length" value="${d4 - elbow_offset - shoulder_offset}" />
-    <xacro:property name="wrist_2_length" value="${d5}" />
-    <xacro:property name="wrist_3_length" value="${d6}" />
+    <!-- <xacro:property name="shoulder_height" value="${0.1273}" /> -->
+    <!-- <xacro:property name="upper_arm_length" value="${0.612}" /> -->
+    <!-- <xacro:property name="forearm_length" value="${0.5723}" /> -->
+    <!-- <xacro:property name="wrist_1_length" value="${0.163941 + 0.1719 - 0.220941}" /> = 0.1149 -->
+    <!-- <xacro:property name="wrist_2_length" value="${0.1157}" /> -->
+    <!-- <xacro:property name="wrist_3_length" value="${0.0922}" /> -->
     <link name="${prefix}base_link" >
       <visual>
@@ -81,5 +83,5 @@
         </geometry>
       </collision>
-      <xacro:cylinder_inertial radius="0.075" length="0.038" mass="${base_mass}">
+      <xacro:cylinder_inertial radius="0.075" length="0.038" mass="4.0">
         <origin xyz="0.0 0.0 0.0" rpy="0 0 0" />
       </xacro:cylinder_inertial>
@@ -88,12 +90,7 @@
       <parent link="${prefix}base_link" />
       <child link = "${prefix}shoulder_link" />
-      <origin xyz="0.0 0.0 ${shoulder_height}" rpy="0.0 0.0 0.0" />
+      <origin xyz="0.0 0.0 0.1273" rpy="0.0 0.0 0.0" />
       <axis xyz="0 0 1" />
-      <xacro:unless value="${joint_limited}">
-        <limit lower="${-2.0 * pi}" upper="${2.0 * pi}" effort="330.0" velocity="2.16"/>
-      </xacro:unless>
-      <xacro:if value="${joint_limited}">
-        <limit lower="${shoulder_pan_lower_limit}" upper="${shoulder_pan_upper_limit}" effort="330.0" velocity="2.16"/>
-      </xacro:if>
+      <limit lower="${shoulder_pan_lower_limit}" upper="${shoulder_pan_upper_limit}" effort="330.0" velocity="2.16"/>
       <dynamics damping="0.0" friction="0.0"/>
     </joint>
@@ -112,5 +109,5 @@
         </geometry>
       </collision>
-      <xacro:cylinder_inertial radius="0.075" length="0.178" mass="${shoulder_mass}">
+      <xacro:cylinder_inertial radius="0.075" length="0.178" mass="7.778">
         <origin xyz="0.0 0.0 0.0" rpy="0 0 0" />
       </xacro:cylinder_inertial>
@@ -119,12 +116,8 @@
       <parent link="${prefix}shoulder_link" />
       <child link = "${prefix}upper_arm_link" />
-      <origin xyz="0.0 ${shoulder_offset} 0.0" rpy="0.0 ${pi / 2.0} 0.0" />
+      <origin xyz="0.0 0.220941 0.0" rpy="0.0 ${pi / 2.0} 0.0" />
       <axis xyz="0 1 0" />
-      <xacro:unless value="${joint_limited}">
-        <limit lower="${-2.0 * pi}" upper="${2.0 * pi}" effort="330.0" velocity="2.16"/>
-      </xacro:unless>
-      <xacro:if value="${joint_limited}">
-        <limit lower="${shoulder_lift_lower_limit}" upper="${shoulder_lift_upper_limit}" effort="330.0" velocity="2.16"/>
-      </xacro:if>
+      <!-- <limit lower="${-2.0 * pi}" upper="${2.0 * pi}" effort="330.0" velocity="2.16"/> -->
+      <limit lower="${shoulder_lift_lower_limit}" upper="${shoulder_lift_upper_limit}" effort="330.0" velocity="2.16"/>
       <dynamics damping="0.0" friction="0.0"/>
     </joint>
@@ -143,6 +136,6 @@
         </geometry>
       </collision>
-      <xacro:cylinder_inertial radius="0.075" length="${-a2}" mass="${upper_arm_mass}">
-        <origin xyz="0.0 0.0 ${-a2/2.0}" rpy="0 0 0" />
+      <xacro:cylinder_inertial radius="0.075" length="${0.612}" mass="12.93">
+        <origin xyz="0.0 0.0 ${0.612/2.0}" rpy="0 0 0" />
       </xacro:cylinder_inertial>
     </link>
@@ -150,12 +143,8 @@
       <parent link="${prefix}upper_arm_link" />
       <child link = "${prefix}forearm_link" />
-      <origin xyz="0.0 ${elbow_offset} ${upper_arm_length}" rpy="0.0 0.0 0.0" />
+      <origin xyz="0.0 -0.1719 0.612" rpy="0.0 0.0 0.0" />
       <axis xyz="0 1 0" />
-      <xacro:unless value="${joint_limited}">
-        <limit lower="${-pi}" upper="${pi}" effort="150.0" velocity="3.15"/>
-      </xacro:unless>
-      <xacro:if value="${joint_limited}">
-        <limit lower="${elbow_joint_lower_limit}" upper="${elbow_joint_upper_limit}" effort="150.0" velocity="3.15"/>
-      </xacro:if>
+      <!-- <limit lower="${-pi}" upper="${pi}" effort="150.0" velocity="3.15"/> -->
+      <limit lower="${elbow_joint_lower_limit}" upper="${elbow_joint_upper_limit}" effort="150.0" velocity="3.15"/>
       <dynamics damping="0.0" friction="0.0"/>
     </joint>
@@ -174,6 +163,6 @@
         </geometry>
       </collision>
-      <xacro:cylinder_inertial radius="0.075" length="${-a3}" mass="${forearm_mass}">
-        <origin xyz="0.0 0.0 ${-a3/2.0}" rpy="0 0 0" />
+      <xacro:cylinder_inertial radius="0.075" length="0.5723" mass="3.87">
+        <origin xyz="0.0 0.0 ${0.5723/2.0}" rpy="0 0 0" />
       </xacro:cylinder_inertial>
     </link>
@@ -181,12 +170,8 @@
       <parent link="${prefix}forearm_link" />
       <child link = "${prefix}wrist_1_link" />
-      <origin xyz="0.0 0.0 ${forearm_length}" rpy="0.0 ${pi / 2.0} 0.0" />
+      <origin xyz="0.0 0.0 0.5723" rpy="0.0 ${pi/2.0} 0.0" />
       <axis xyz="0 1 0" />
-      <xacro:unless value="${joint_limited}">
-        <limit lower="${-2.0 * pi}" upper="${2.0 * pi}" effort="54.0" velocity="3.2"/>
-      </xacro:unless>
-      <xacro:if value="${joint_limited}">
-        <limit lower="${wrist_1_lower_limit}" upper="${wrist_1_upper_limit}" effort="54.0" velocity="3.2"/>
-      </xacro:if>
+      <!-- <limit lower="${-2.0 * pi}" upper="${2.0 * pi}" effort="54.0" velocity="3.2"/> -->
+      <limit lower="${wrist_1_lower_limit}" upper="${wrist_1_upper_limit}" effort="54.0" velocity="3.2"/>
       <dynamics damping="0.0" friction="0.0"/>
     </joint>
@@ -205,5 +190,5 @@
         </geometry>
       </collision>
-      <xacro:cylinder_inertial radius="0.075" length="0.12" mass="${wrist_1_mass}">
+      <xacro:cylinder_inertial radius="0.075" length="0.12" mass="1.96">
         <origin xyz="0.0 0.0 0.0" rpy="0 0 0" />
       </xacro:cylinder_inertial>
@@ -212,12 +197,8 @@
       <parent link="${prefix}wrist_1_link" />
       <child link = "${prefix}wrist_2_link" />
-      <origin xyz="0.0 ${wrist_1_length} 0.0" rpy="0.0 0.0 0.0" />
+      <origin xyz="0.0 0.1149 0.0" rpy="0.0 0.0 0.0" />
       <axis xyz="0 0 1" />
-      <xacro:unless value="${joint_limited}">
-        <limit lower="${-2.0 * pi}" upper="${2.0 * pi}" effort="54.0" velocity="3.2"/>
-      </xacro:unless>
-      <xacro:if value="${joint_limited}">
-        <limit lower="${wrist_2_lower_limit}" upper="${wrist_2_upper_limit}" effort="54.0" velocity="3.2"/>
-      </xacro:if>
+      <!-- <limit lower="${-2.0 * pi}" upper="${2.0 * pi}" effort="54.0" velocity="3.2"/> -->
+      <limit lower="${wrist_2_lower_limit}" upper="${wrist_2_upper_limit}" effort="54.0" velocity="3.2"/>
       <dynamics damping="0.0" friction="0.0"/>
     </joint>
@@ -236,5 +217,5 @@
         </geometry>
       </collision>
-      <xacro:cylinder_inertial radius="0.075" length="0.12" mass="${wrist_2_mass}">
+      <xacro:cylinder_inertial radius="0.075" length="0.12" mass="1.96">
         <origin xyz="0.0 0.0 0.0" rpy="0 0 0" />
       </xacro:cylinder_inertial>
@@ -243,12 +224,8 @@
       <parent link="${prefix}wrist_2_link" />
       <child link = "${prefix}wrist_3_link" />
-      <origin xyz="0.0 0.0 ${wrist_2_length}" rpy="0.0 0.0 0.0" />
+      <origin xyz="0.0 0.0 0.1157" rpy="0.0 0.0 0.0" />
       <axis xyz="0 1 0" />
-      <xacro:unless value="${joint_limited}">
-        <limit lower="${-2.0 * pi}" upper="${2.0 * pi}" effort="54.0" velocity="3.2"/>
-      </xacro:unless>
-      <xacro:if value="${joint_limited}">
-        <limit lower="${wrist_3_lower_limit}" upper="${wrist_3_upper_limit}" effort="54.0" velocity="3.2"/>
-      </xacro:if>
+      <!-- <limit lower="${-2.0 * pi}" upper="${2.0 * pi}" effort="54.0" velocity="3.2"/> -->
+      <limit lower="${wrist_3_lower_limit}" upper="${wrist_3_upper_limit}" effort="54.0" velocity="3.2"/>
       <dynamics damping="0.0" friction="0.0"/>
     </joint>
@@ -267,5 +244,5 @@
         </geometry>
       </collision>
-      <xacro:cylinder_inertial radius="0.075" length="0.12" mass="${wrist_3_mass}">
+      <xacro:cylinder_inertial radius="0.075" length="0.12" mass="0.202">
         <origin xyz="0.0 0.0 0.0" rpy="0 0 0" />
       </xacro:cylinder_inertial>
@@ -274,5 +251,5 @@
       <parent link="${prefix}wrist_3_link" />
       <child link = "${prefix}ee_link" />
-      <origin xyz="0.0 ${wrist_3_length} 0.0" rpy="0.0 0.0 ${pi/2.0}" />
+      <origin xyz="0.0 0.0922 0.0" rpy="0.0 0.0 ${pi/2.0}" />
     </joint>
     <link name="${prefix}ee_link">
@@ -408,10 +385,5 @@
       <origin xyz="0.05 0.0 0.05" rpy="0.0 0.0 0.0" />
       <axis xyz="0 0 1" />
-      <xacro:unless value="${joint_limited}">
-        <limit lower="${-2.0 * pi}" upper="${2.0 * pi}" effort="54.0" velocity="3.2"/>
-      </xacro:unless>
-      <xacro:if value="${joint_limited}">
-        <limit lower="${hand_lower_limit}" upper="${hand_upper_limit}" effort="54.0" velocity="3.2"/>
-      </xacro:if>
+      <limit lower="${hand_lower_limit}" upper="${hand_upper_limit}" effort="54.0" velocity="3.2"/>
       <dynamics damping="0.0" friction="0.0"/>
     </joint> -->
@@ -446,10 +418,5 @@
   <origin xyz="0.0 0.0 -0.25" rpy="0.0 0.0 0.0" />
   <axis xyz="0 0 1" />
-  <xacro:unless value="${joint_limited}">
-    <limit lower="${-2.0 * pi}" upper="${2.0 * pi}" effort="54.0" velocity="3.2"/>
-  </xacro:unless>
-  <xacro:if value="${joint_limited}">
-    <limit lower="${forearm_lower_limit}" upper="${forearm_upper_limit}" effort="54.0" velocity="3.2"/>
-  </xacro:if>
+  <limit lower="${forearm_lower_limit}" upper="${forearm_upper_limit}" effort="54.0" velocity="3.2"/>
   <dynamics damping="0.0" friction="0.0"/>
 </joint>
@@ -522,10 +489,5 @@
       <origin xyz="0.0 0.0 0.0" rpy="0.0 0.0 0.0" />
       <axis xyz="0 0 1" />
-      <xacro:unless value="${joint_limited}">
-        <limit lower="${-2.0 * pi}" upper="${2.0 * pi}" effort="54.0" velocity="3.2"/>
-      </xacro:unless>
-      <xacro:if value="${joint_limited}">
-        <limit lower="${arm_elbow_lower_limit}" upper="${arm_elbow_upper_limit}" effort="54.0" velocity="3.2"/>
-      </xacro:if>
+      <limit lower="${arm_elbow_lower_limit}" upper="${arm_elbow_upper_limit}" effort="54.0" velocity="3.2"/>
       <dynamics damping="0.0" friction="0.0"/>
     </joint>
@@ -552,10 +514,5 @@
       <origin xyz="0.15 0.0 0.0" rpy="0.0 0.0 0.0" />
       <axis xyz="0 0 1" />
-      <xacro:unless value="${joint_limited}">
-        <limit lower="${-2.0 * pi}" upper="${2.0 * pi}" effort="54.0" velocity="3.2"/>
-      </xacro:unless>
-      <xacro:if value="${joint_limited}">
-        <limit lower="${arm_forearm_lower_limit}" upper="${arm_forearm_upper_limit}" effort="54.0" velocity="3.2"/>
-      </xacro:if>
+      <limit lower="${arm_forearm_lower_limit}" upper="${arm_forearm_upper_limit}" effort="54.0" velocity="3.2"/>
       <dynamics damping="0.0" friction="0.0"/>
     </joint>
@@ -582,10 +539,5 @@
       <origin xyz="0.15 0.0 0.0" rpy="0.0 0.0 0.0" />
       <axis xyz="0 0 1" />
-      <xacro:unless value="${joint_limited}">
-        <limit lower="${-2.0 * pi}" upper="${2.0 * pi}" effort="54.0" velocity="3.2"/>
-      </xacro:unless>
-      <xacro:if value="${joint_limited}">
-        <limit lower="${arm_wrist_lower_limit}" upper="${arm_wrist_upper_limit}" effort="54.0" velocity="3.2"/>
-      </xacro:if>
+      <limit lower="${arm_wrist_lower_limit}" upper="${arm_wrist_upper_limit}" effort="54.0" velocity="3.2"/>
       <dynamics damping="0.0" friction="0.0"/>
     </joint> -->
@@ -604,10 +556,10 @@
     </joint>
     <!-- Frame coincident with all-zeros TCP on UR controller -->
-    <link name="${prefix}tool0"/>
+    <!-- <link name="${prefix}tool0"/>
     <joint name="${prefix}wrist_3_link-tool0_fixed_joint" type="fixed">
-      <origin xyz="0 ${wrist_3_length} 0" rpy="${pi/-2.0} 0 0"/>
+      <origin xyz="0 0.0922 0" rpy="${pi/-2.0} 0 0"/>
       <parent link="${prefix}wrist_3_link"/>
       <child link="${prefix}tool0"/>
-    </joint>
+    </joint> -->
   </xacro:macro>
 </robot>

File: src/universal_robot/ur_description/urdf/ur10_joint_limited_robot.urdf.xacro (robot description, xacro)
@@ -5,5 +5,5 @@
   <xacro:include filename="$(find ur_description)/urdf/common.gazebo.xacro" />
   <!-- ur10 -->
-  <xacro:include filename="$(find ur_description)/urdf/ur10.urdf.xacro" />
+  <xacro:include filename="$(find ur_description)/urdf/Sur10.urdf.xacro" />
   <!-- arm -->
   <xacro:ur10_robot prefix="" joint_limited="true"
