Commit message: Added Sur10.urdf.xacro - 3 DOF and 4 DOF human arm

File: src/universal_robot/ur_description/urdf/Sur10.urdf.xacro (robot description, xacro)
@@ -27,4 +27,12 @@
      hand_lower_limit:=${-pi}    hand_upper_limit:=${pi}
      ">
+     <!-- shoulder_pan_lower_limit:=${-pi}    shoulder_pan_upper_limit:=${pi}
+    shoulder_lift_lower_limit:=${-pi}    shoulder_lift_upper_limit:=${pi}
+    elbow_joint_lower_limit:=${-pi}    elbow_joint_upper_limit:=${pi}
+    wrist_1_lower_limit:=${-pi}    wrist_1_upper_limit:=${pi}
+    wrist_2_lower_limit:=${-pi}    wrist_2_upper_limit:=${pi}
+    wrist_3_lower_limit:=${-pi}    wrist_3_upper_limit:=${pi}
+     wrist_3_lower_limit:=${-pi}    wrist_3_upper_limit:=${pi}
+     hand_lower_limit:=${-pi}    hand_upper_limit:=${pi} -->
      <!-- arm_elbow_lower_limit:=${-pi}    arm_elbow_upper_limit:=${pi}
      arm_forearm_lower_limit:=${-pi}    arm_forearm_upper_limit:=${pi}
@@ -45,10 +53,10 @@
         The permutation was guessed by looking at the UR5 parameters.
         Serious use of these parameters needs further inspection. -->
-    <xacro:property name="shoulder_cog" value="0.00008 0.00244 -0.037" />
+    <!-- <xacro:property name="shoulder_cog" value="0.00008 0.00244 -0.037" />
     <xacro:property name="upper_arm_cog" value="0.00001 0.15061 0.38757" />
     <xacro:property name="forearm_cog" value="-0.00012 0.06112 0.1984" />
     <xacro:property name="wrist_1_cog" value="-0.00021 -0.00112 0.02269" />
     <xacro:property name="wrist_2_cog" value="-0.00021 0.00112 0.002269" />
-    <xacro:property name="wrist_3_cog" value="0 -0.001156 -0.00149" />
+    <xacro:property name="wrist_3_cog" value="0 -0.001156 -0.00149" /> -->
     <!-- Kinematic model -->
     <!-- Properties from urcontrol.conf -->
@@ -69,5 +77,5 @@
     <!-- <xacro:property name="wrist_2_length" value="${0.1157}" /> -->
     <!-- <xacro:property name="wrist_3_length" value="${0.0922}" /> -->
-    <link name="${prefix}base_link" >
+    <link name="base_link" >
       <visual>
         <geometry>
@@ -87,13 +95,13 @@
       </xacro:cylinder_inertial>
     </link>
-    <joint name="${prefix}shoulder_pan_joint" type="revolute">
-      <parent link="${prefix}base_link" />
-      <child link = "${prefix}shoulder_link" />
+    <joint name="shoulder_pan_joint" type="revolute">
+      <parent link="base_link" />
+      <child link = "shoulder_link" />
       <origin xyz="0.0 0.0 0.1273" rpy="0.0 0.0 0.0" />
       <axis xyz="0 0 1" />
-      <limit lower="${shoulder_pan_lower_limit}" upper="${shoulder_pan_upper_limit}" effort="330.0" velocity="2.16"/>
-      <dynamics damping="0.0" friction="0.0"/>
-    </joint>
-    <link name="${prefix}shoulder_link">
+      <limit lower="0" upper="1.5070796" effort="330.0" velocity="2.16"/>
+      <dynamics damping="0.0" friction="0.0"/>
+    </joint>
+    <link name="shoulder_link">
       <visual>
         <geometry>
@@ -113,14 +121,14 @@
       </xacro:cylinder_inertial>
     </link>
-    <joint name="${prefix}shoulder_lift_joint" type="revolute">
-      <parent link="${prefix}shoulder_link" />
-      <child link = "${prefix}upper_arm_link" />
+    <joint name="shoulder_lift_joint" type="revolute">
+      <parent link="shoulder_link" />
+      <child link = "upper_arm_link" />
       <origin xyz="0.0 0.220941 0.0" rpy="0.0 ${pi / 2.0} 0.0" />
       <axis xyz="0 1 0" />
       <!-- <limit lower="${-2.0 * pi}" upper="${2.0 * pi}" effort="330.0" velocity="2.16"/> -->
-      <limit lower="${shoulder_lift_lower_limit}" upper="${shoulder_lift_upper_limit}" effort="330.0" velocity="2.16"/>
-      <dynamics damping="0.0" friction="0.0"/>
-    </joint>
-    <link name="${prefix}upper_arm_link">
+      <limit lower="-3.14159265" upper="0" effort="330.0" velocity="2.16"/>
+      <dynamics damping="0.0" friction="0.0"/>
+    </joint>
+    <link name="upper_arm_link">
       <visual>
         <geometry>
@@ -140,14 +148,14 @@
       </xacro:cylinder_inertial>
     </link>
-    <joint name="${prefix}elbow_joint" type="revolute">
-      <parent link="${prefix}upper_arm_link" />
-      <child link = "${prefix}forearm_link" />
+    <joint name="elbow_joint" type="revolute">
+      <parent link="upper_arm_link" />
+      <child link = "forearm_link" />
       <origin xyz="0.0 -0.1719 0.612" rpy="0.0 0.0 0.0" />
       <axis xyz="0 1 0" />
       <!-- <limit lower="${-pi}" upper="${pi}" effort="150.0" velocity="3.15"/> -->
-      <limit lower="${elbow_joint_lower_limit}" upper="${elbow_joint_upper_limit}" effort="150.0" velocity="3.15"/>
-      <dynamics damping="0.0" friction="0.0"/>
-    </joint>
-    <link name="${prefix}forearm_link">
+      <limit lower="0" upper="3.14159265" effort="150.0" velocity="3.15"/>
+      <dynamics damping="0.0" friction="0.0"/>
+    </joint>
+    <link name="forearm_link">
       <visual>
          <geometry>
@@ -167,14 +175,14 @@
       </xacro:cylinder_inertial>
     </link>
-    <joint name="${prefix}wrist_1_joint" type="revolute">
-      <parent link="${prefix}forearm_link" />
-      <child link = "${prefix}wrist_1_link" />
+    <joint name="wrist_1_joint" type="revolute">
+      <parent link="forearm_link" />
+      <child link = "wrist_1_link" />
       <origin xyz="0.0 0.0 0.5723" rpy="0.0 ${pi/2.0} 0.0" />
       <axis xyz="0 1 0" />
       <!-- <limit lower="${-2.0 * pi}" upper="${2.0 * pi}" effort="54.0" velocity="3.2"/> -->
-      <limit lower="${wrist_1_lower_limit}" upper="${wrist_1_upper_limit}" effort="54.0" velocity="3.2"/>
-      <dynamics damping="0.0" friction="0.0"/>
-    </joint>
-    <link name="${prefix}wrist_1_link">
+      <limit lower="-3.14159265" upper="0" effort="54.0" velocity="3.2"/>
+      <dynamics damping="0.0" friction="0.0"/>
+    </joint>
+    <link name="wrist_1_link">
       <visual>
         <geometry>
@@ -194,14 +202,14 @@
       </xacro:cylinder_inertial>
     </link>
-    <joint name="${prefix}wrist_2_joint" type="revolute">
-      <parent link="${prefix}wrist_1_link" />
-      <child link = "${prefix}wrist_2_link" />
+    <joint name="wrist_2_joint" type="revolute">
+      <parent link="wrist_1_link" />
+      <child link = "wrist_2_link" />
       <origin xyz="0.0 0.1149 0.0" rpy="0.0 0.0 0.0" />
       <axis xyz="0 0 1" />
       <!-- <limit lower="${-2.0 * pi}" upper="${2.0 * pi}" effort="54.0" velocity="3.2"/> -->
-      <limit lower="${wrist_2_lower_limit}" upper="${wrist_2_upper_limit}" effort="54.0" velocity="3.2"/>
-      <dynamics damping="0.0" friction="0.0"/>
-    </joint>
-    <link name="${prefix}wrist_2_link">
+      <limit lower="-3.14159265" upper="0.785398" effort="54.0" velocity="3.2"/>
+      <dynamics damping="0.0" friction="0.0"/>
+    </joint>
+    <link name="wrist_2_link">
       <visual>
         <geometry>
@@ -221,14 +229,14 @@
       </xacro:cylinder_inertial>
     </link>
-    <joint name="${prefix}wrist_3_joint" type="revolute">
-      <parent link="${prefix}wrist_2_link" />
-      <child link = "${prefix}wrist_3_link" />
+    <joint name="wrist_3_joint" type="revolute">
+      <parent link="wrist_2_link" />
+      <child link = "wrist_3_link" />
       <origin xyz="0.0 0.0 0.1157" rpy="0.0 0.0 0.0" />
       <axis xyz="0 1 0" />
       <!-- <limit lower="${-2.0 * pi}" upper="${2.0 * pi}" effort="54.0" velocity="3.2"/> -->
-      <limit lower="${wrist_3_lower_limit}" upper="${wrist_3_upper_limit}" effort="54.0" velocity="3.2"/>
-      <dynamics damping="0.0" friction="0.0"/>
-    </joint>
-    <link name="${prefix}wrist_3_link">
+      <limit lower="-3.14159265" upper="3.14159265" effort="54.0" velocity="3.2"/>
+      <dynamics damping="0.0" friction="0.0"/>
+    </joint>
+    <link name="wrist_3_link">
       <visual>
         <geometry>
@@ -248,10 +256,10 @@
       </xacro:cylinder_inertial>
     </link>
-    <joint name="${prefix}ee_fixed_joint" type="fixed">
-      <parent link="${prefix}wrist_3_link" />
-      <child link = "${prefix}ee_link" />
+    <joint name="ee_fixed_joint" type="fixed">
+      <parent link="wrist_3_link" />
+      <child link = "ee_link" />
       <origin xyz="0.0 0.0922 0.0" rpy="0.0 0.0 ${pi/2.0}" />
     </joint>
-    <link name="${prefix}ee_link">
+    <link name="ee_link">
       <collision>
         <geometry>
@@ -261,15 +269,15 @@
       </collision>
     </link>
-    <joint name="${prefix}ee_plate_joint" type="fixed">
-      <parent link="${prefix}ee_link" />
-      <child link = "${prefix}ee_metal_plate" />
+    <joint name="ee_plate_joint" type="fixed">
+      <parent link="ee_link" />
+      <child link = "ee_metal_plate" />
       <origin xyz="0.0 0.0 0.0" rpy="0.0 0.0 0.0" />
     </joint>
-    <link name="${prefix}ee_metal_plate">
+    <link name="ee_metal_plate">
       <visual>
         <geometry>
           <box size="0.085 0.085 0.01"/>
         </geometry>
-        <origin rpy="0 ${pi/2.0} 0" xyz="0 0 0"/>
+        <origin rpy="0 1.570796 0" xyz="0 0 0"/>
         <material name="LightGrey">
           <color rgba="0.7 0.7 0.7 1.0"/>
@@ -280,18 +288,18 @@
           <box size="0.085 0.085 0.01"/>
         </geometry>
-        <origin rpy="0 ${pi/2.0} 0" xyz="0 0 0"/>
-      </collision>
-    </link>
-    <joint name="${prefix}ee_sensor_joint" type="fixed">
-      <parent link="${prefix}ee_metal_plate" />
-      <child link = "${prefix}ee_sensor_plate" />
+        <origin rpy="0 1.570796 0" xyz="0 0 0"/>
+      </collision>
+    </link>
+    <joint name="ee_sensor_joint" type="fixed">
+      <parent link="ee_metal_plate" />
+      <child link = "ee_sensor_plate" />
       <origin xyz="0.022 0.0 0.0" rpy="0.0 0.0 0.0" />
     </joint>
-    <link name="${prefix}ee_sensor_plate">
+    <link name="ee_sensor_plate">
       <visual>
         <geometry>
           <cylinder length="0.035" radius="0.06"/>
         </geometry>
-        <origin rpy="0 ${pi/2.0} 0" xyz="0 0 0"/>
+        <origin rpy="0 1.570796 0" xyz="0 0 0"/>
         <material name="Black">
           <color rgba="0.0 0.0 0.0 1.0"/>
@@ -302,18 +310,18 @@
           <cylinder length="0.035" radius="0.06"/>
         </geometry>
-        <origin rpy="0 ${pi/2.0} 0" xyz="0 0 0"/>
-      </collision>
-    </link>
-    <joint name="${prefix}ee_magnet_joint" type="fixed">
-      <parent link="${prefix}ee_sensor_plate" />
-      <child link = "${prefix}ee_magnet_cylinder" />
+        <origin rpy="0 1.570796 0" xyz="0 0 0"/>
+      </collision>
+    </link>
+    <joint name="ee_magnet_joint" type="fixed">
+      <parent link="ee_sensor_plate" />
+      <child link = "ee_magnet_cylinder" />
       <origin xyz="0.042 0.0 0.0" rpy="0.0 0.0 0.0" />
     </joint>
-    <link name="${prefix}ee_magnet_cylinder">
+    <link name="ee_magnet_cylinder">
       <visual>
         <geometry>
           <cylinder length="0.05" radius="0.04"/>
         </geometry>
-        <origin rpy="0 ${pi/2.0} 0" xyz="0 0 0"/>
+        <origin rpy="0 1.570796 0" xyz="0 0 0"/>
         <material name="White">
           <color rgba="1.0 1.0 1.0 1.0"/>
@@ -324,5 +332,5 @@
           <cylinder length="0.05" radius="0.04"/>
         </geometry>
-        <origin rpy="0 ${pi/2.0} 0" xyz="0 0 0"/>
+        <origin rpy="0 1.570796 0" xyz="0 0 0"/>
       </collision>
     </link>
@@ -353,10 +361,10 @@
       </collision>
     </link> -->
-    <joint name="${prefix}fake_arm_joint" type="fixed">
-      <parent link="${prefix}ee_magnet_cylinder" />
-      <child link = "${prefix}fake_arm_link" />
+    <!-- <joint name="fake_arm_joint" type="fixed">
+      <parent link="ee_magnet_cylinder" />
+      <child link = "fake_arm_link" />
       <origin xyz="0.05 0.0 -0.12" rpy="0.0 0.0 0.0" />
     </joint>
-    <link name="${prefix}fake_arm_link">
+    <link name="fake_arm_link">
       <visual>
         <geometry>
@@ -374,8 +382,8 @@
         <origin rpy="0 0 0" xyz="0 0 0"/>
       </collision>
-    </link>
-    <joint name="${prefix}fake_hand_joint" type="fixed">
-      <parent link="${prefix}ee_magnet_cylinder" />
-      <child link = "${prefix}fake_hand_link" />
+    </link> -->
+    <joint name="fake_hand_joint" type="fixed">
+      <parent link="ee_magnet_cylinder" />
+      <child link = "fake_hand_link" />
       <origin xyz="0.05 0.0 0.05" rpy="0.0 0.0 0.0" />
     </joint>
@@ -388,5 +396,5 @@
       <dynamics damping="0.0" friction="0.0"/>
     </joint> -->
-    <link name="${prefix}fake_hand_link">
+    <link name="fake_hand_link">
       <visual>
         <geometry>
@@ -394,5 +402,5 @@
           <box size="0.1 0.05 0.05"/>
         </geometry>
-        <origin rpy="0 ${pi/2.0} 0" xyz="0 0 0"/>
+        <origin rpy="0 1.570796 0" xyz="0 0 0"/>
         <material name="HandColor">
           <color rgba="0.4 0.4 0.4 1.0"/>
@@ -404,8 +412,157 @@
           <box size="0.1 0.05 0.05"/>
         </geometry>
-        <origin rpy="0 ${pi/2.0} 0" xyz="0 0 0"/>
+        <origin rpy="0 1.570796 0" xyz="0 0 0"/>
       </collision>
     </link>
 <!-- #########################ARM TEST########################## -->
+<joint name="arm_base_joint" type="fixed">
+  <parent link="base_link" />
+  <child link = "arm_shoulder_1_link" />
+  <origin xyz="-0.2 0.5 0.35" rpy="0.0 0.0 0.0" />
+</joint>
+<link name="arm_shoulder_1_link">
+  <visual>
+    <geometry>
+      <box size="0.07 0.07 0.1"/>
+    </geometry>
+    <origin rpy="0 0 0" xyz="0 0 0"/>
+    <material name="ShoulderColour">
+      <color rgba="0.4 0.4 0.4 1.0"/>
+    </material>
+  </visual>
+  <collision>
+    <geometry>
+      <box size="0.05 0.05 0.05"/>
+    </geometry>
+    <origin rpy="0 0 0" xyz="0 0 0"/>
+  </collision>
+</link>
+<joint name="arm_shoulder_1_joint" type="revolute">
+  <parent link="arm_shoulder_1_link" />
+  <child link = "arm_shoulder_2_link" />
+  <origin xyz="0.0 0.0 0.0" rpy="0.0 0.0 0.0" />
+  <axis xyz="0 1 0" />
+  <limit lower="-3.14159265" upper="3.14159265" effort="54.0" velocity="3.2"/>
+  <dynamics damping="0.0" friction="0.0"/>
+</joint>
+<link name="arm_shoulder_2_link">
+  <visual>
+    <geometry>
+      <box size="0.01 0.01 0.01"/>
+    </geometry>
+    <origin rpy="0 0 0" xyz="0 0 0"/>
+    <material name="ShoulderColour">
+      <color rgba="0.4 0.4 0.4 1.0"/>
+    </material>
+  </visual>
+  <collision>
+    <geometry>
+      <box size="0.01 0.01 0.01"/>
+    </geometry>
+    <origin rpy="0 0 0" xyz="0 0 0"/>
+  </collision>
+</link>
+<joint name="arm_shoulder_2_joint" type="revolute">
+  <parent link="arm_shoulder_2_link" />
+  <child link = "arm_upper_arm_link" />
+  <origin xyz="0.0 0.0 0.0" rpy="0.0 0.0 0.0" />
+  <axis xyz="0 0 1" />
+  <limit lower="-3.14159265" upper="3.14159265" effort="54.0" velocity="3.2"/>
+  <dynamics damping="0.0" friction="0.0"/>
+</joint>
+<link name="arm_upper_arm_link">
+  <visual>
+    <geometry>
+      <cylinder length="0.3" radius="0.035"/>
+    </geometry>
+    <origin rpy="0 1.570796 0" xyz="0.15 0 0"/>
+    <material name="Elbow">
+      <color rgba="0.2 0.2 0.2 1.0"/>
+    </material>
+  </visual>
+  <collision>
+    <geometry>
+      <cylinder length="0.3" radius="0.035"/>
+    </geometry>
+    <origin rpy="0 1.570796 0" xyz="0.15 0 0"/>
+  </collision>
+</link>
+<joint name="arm_elbow_1_joint" type="revolute">
+  <parent link="arm_upper_arm_link" />
+  <child link = "arm_forearm_1_link" />
+  <origin xyz="0.3 0.0 0.0" rpy="0.0 0.0 0.0" />
+  <axis xyz="0 0 1" />
+  <limit lower="-3.14159265" upper="3.14159265" effort="54.0" velocity="3.2"/>
+  <dynamics damping="0.0" friction="0.0"/>
+</joint>
+<link name="arm_forearm_1_link">
+  <visual>
+    <geometry>
+      <box size="0.01 0.01 0.01"/>
+    </geometry>
+    <origin rpy="0 1.570796 0" xyz="0.0 0.0 0.0"/>
+    <material name="FA">
+      <color rgba="0.0 0.0 0.0 1.0"/>
+    </material>
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
File: src/universal_robot/ur_description/urdf/human_arm_3dof.urdf (robot description, URDF)
Before this commit: robot ur10, 6 links, 5 joints
Links:
- removed link arm_forearm_2_link
- link arm_forearm_1_link: geometry collision cylinder length=0.25 radius=0.025; visual cylinder length=0.25 radius=0.025
- link arm_shoulder_2_link: geometry collision box size=0.05 0.05 0.05; visual box size=0.01 0.01 0.01
Joints:
- removed joint arm_elbow_2_joint

File: src/universal_robot/ur_description/urdf/ur10.urdf.xacro (robot description, xacro)
@@ -590,6 +590,6 @@
       <dynamics damping="0.0" friction="0.0"/>
     </joint> -->
-    <!-- <xacro:ur_arm_transmission prefix="${prefix}" />
-    <xacro:ur_arm_gazebo prefix="${prefix}" /> -->
+    <xacro:ur_arm_transmission prefix="${prefix}" />
+    <xacro:ur_arm_gazebo prefix="${prefix}" />
     <!-- ROS base_link to UR 'Base' Coordinates transform -->
     <link name="${prefix}base"/>

File: src/universal_robot/ur_description/urdf/ur10_joint_limited_robot.urdf.xacro (robot description, xacro)
@@ -3,6 +3,7 @@
        name="ur10" >
   <!-- common stuff -->
-  <xacro:include filename="$(find ur_description)/urdf/common.gazebo.xacro" />
+  <!-- <xacro:include filename="$(find ur_description)/urdf/common.gazebo.xacro" /> -->
   <!-- ur10 -->
+  <!-- <xacro:include filename="$(find ur_description)/urdf/ur10.urdf.xacro" /> -->
   <xacro:include filename="$(find ur_description)/urdf/Sur10.urdf.xacro" />
   <!-- arm -->

Commit message: Added gazePoint service. Managed to get arm to be the end effector

File: src/universal_robot/ur_description/urdf/Sur10.urdf.xacro (robot description, xacro)
@@ -540,4 +540,34 @@
       <cylinder length="0.25" radius="0.025"/>
     </geometry>
+    <origin rpy="0 1.570796 0" xyz="0.125 0.0 0.0"/>
+  </collision>
+  <!-- <inertial>
+    <mass value="1.80"/>
+    <inertia ixx="0.4" ixy="0.0" ixz="0.0" iyy="0.4" iyz="0.0" izz="0.2"/>
+    <origin xyz="0.0 0.0 0.0" rpy="0 0 0" />
+  </inertial> -->
+</link>
+<joint name="arm_ee_joint" type="fixed">
+  <parent link="arm_forearm_2_link" />
+  <child link = "arm_ee_link" />
+  <origin xyz="0.25 0.0 0.0" rpy="0.0 0.0 0.0" />
+  <!-- <axis xyz="0 1 0" /> -->
+  <!-- <limit lower="-3.14159265" upper="3.14159265" effort="54.0" velocity="3.2"/> -->
+  <!-- <dynamics damping="0.0" friction="0.0"/> -->
+</joint>
+<link name="arm_ee_link">
+  <visual>
+    <geometry>
+      <box size="0.05 0.05 0.05"/>
+    </geometry>
+    <origin rpy="0 1.570796 0" xyz="0.0 0.0 0.0"/>
+    <material name="FAee">
+      <color rgba="0.0 0.0 1.0 1.0"/>
+    </material>
+  </visual>
+  <collision>
+    <geometry>
+      <box size="0.05 0.05 0.05"/>
+    </geometry>
     <origin rpy="0 1.570796 0" xyz="0.0 0.0 0.0"/>
   </collision>
@@ -556,4 +586,5 @@
   <dynamics damping="0.0" friction="0.0"/>
 </joint> -->
+<!--
 <joint name="arm_common_joint" type="fixed">
   <parent link="arm_forearm_2_link" />
@@ -563,5 +594,5 @@
   <limit lower="-3.14159265" upper="3.14159265" effort="54.0" velocity="3.2"/>
   <dynamics damping="0.0" friction="0.0"/>
-</joint>
+</joint> -->
 <!-- ##################### -->
 <!-- <joint name="${prefix}fake_forearm_joint" type="fixed">

File: src/universal_robot/ur_description/urdf/ur10_joint_limited_robot.urdf.xacro (robot description, xacro)
@@ -5,6 +5,6 @@
   <!-- <xacro:include filename="$(find ur_description)/urdf/common.gazebo.xacro" /> -->
   <!-- ur10 -->
-  <xacro:include filename="$(find ur_description)/urdf/ur10.urdf.xacro" />
-  <!-- <xacro:include filename="$(find ur_description)/urdf/Sur10.urdf.xacro" /> -->
+  <!-- <xacro:include filename="$(find ur_description)/urdf/ur10.urdf.xacro" /> -->
+  <xacro:include filename="$(find ur_description)/urdf/Sur10.urdf.xacro" />
   <!-- arm -->
   <xacro:ur10_robot prefix="" joint_limited="true"
