Commit message: Gaze integration, moved all objects to moveit python, fake gaze publisher

File: src/universal_robot/ur_description/urdf/ur10.urdf.xacro (robot description, xacro)
@@ -342,14 +342,17 @@
       </collision>
     </link>
+<!--
     <joint name="${prefix}fake_hand_joint" type="fixed">
       <parent link="${prefix}ee_magnet_cylinder" />
       <child link = "${prefix}fake_hand_link" />
-      <origin xyz="0.0 0.0 0.065" rpy="0.0 0.0 0.0" />
-    </joint>
-    <link name="${prefix}fake_hand_link">
-      <visual>
-        <geometry>
-          <box size="0.08 0.05 0.05"/>
-        </geometry>
+      <origin xyz="0.05 0.0 -0.05" rpy="0.0 0.0 0.0" /> -->
+      <!-- <origin xyz="0.0 0.0 0.065" rpy="0.0 0.0 0.0" /> -->
+    <!-- </joint> -->
+    <!-- <link name="${prefix}fake_hand_link">
+      <visual>
+        <geometry>
+          <box size="0.35 0.05 0.05"/> -->
+          <!-- <box size="0.08 0.05 0.05"/> -->
+        <!-- </geometry>
         <origin rpy="0 ${pi/2.0} 0" xyz="0 0 0"/>
         <material name="HandColor">
@@ -359,5 +362,53 @@
       <collision>
         <geometry>
-          <box size="0.08 0.05 0.05"/>
+          <box size="0.35 0.05 0.05"/> -->
+          <!-- <box size="0.08 0.05 0.05"/> -->
+        <!-- </geometry>
+        <origin rpy="0 ${pi/2.0} 0" xyz="0 0 0"/>
+      </collision>
+    </link> -->
+    <joint name="${prefix}fake_arm_joint" type="fixed">
+      <parent link="${prefix}ee_magnet_cylinder" />
+      <child link = "${prefix}fake_arm_link" />
+      <origin xyz="0.05 0.0 -0.12" rpy="0.0 0.0 0.0" />
+    </joint>
+    <link name="${prefix}fake_arm_link">
+      <visual>
+        <geometry>
+          <cylinder length="0.25" radius="0.025"/>
+        </geometry>
+        <origin rpy="0 0 0" xyz="0 0 0"/>
+        <material name="ArmColor">
+          <color rgba="1.0 1.0 1.0 1.0"/>
+        </material>
+      </visual>
+      <collision>
+        <geometry>
+          <cylinder length="0.25" radius="0.025"/>
+        </geometry>
+        <origin rpy="0 0 0" xyz="0 0 0"/>
+      </collision>
+    </link>
+    <joint name="${prefix}fake_hand_joint" type="fixed">
+      <parent link="${prefix}ee_magnet_cylinder" />
+      <child link = "${prefix}fake_hand_link" />
+      <origin xyz="0.05 0.0 0.05" rpy="0.0 0.0 0.0" />
+      <!-- <origin xyz="0.0 0.0 0.065" rpy="0.0 0.0 0.0" /> -->
+    </joint>
+    <link name="${prefix}fake_hand_link">
+      <visual>
+        <geometry>
+          <!-- <box size="0.35 0.05 0.05"/> -->
+          <box size="0.1 0.05 0.05"/>
+        </geometry>
+        <origin rpy="0 ${pi/2.0} 0" xyz="0 0 0"/>
+        <material name="HandColor">
+          <color rgba="0.4 0.4 0.4 1.0"/>
+        </material>
+      </visual>
+      <collision>
+        <geometry>
+          <!-- <box size="0.35 0.05 0.05"/> -->
+          <box size="0.1 0.05 0.05"/>
         </geometry>
         <origin rpy="0 ${pi/2.0} 0" xyz="0 0 0"/>

Commit message: Pose to target object

File: src/universal_robot/ur_description/urdf/ur10.urdf.xacro (robot description, xacro)
@@ -22,5 +22,13 @@
 		 wrist_1_lower_limit:=${-pi}    wrist_1_upper_limit:=${pi}
 		 wrist_2_lower_limit:=${-pi}    wrist_2_upper_limit:=${pi}
-		 wrist_3_lower_limit:=${-pi}    wrist_3_upper_limit:=${pi}">
+		 wrist_3_lower_limit:=${-pi}    wrist_3_upper_limit:=${pi}
+     wrist_3_lower_limit:=${-pi}    wrist_3_upper_limit:=${pi}
+     hand_lower_limit:=${-pi}    hand_upper_limit:=${pi}
+     ">
+     <!-- arm_elbow_lower_limit:=${-pi}    arm_elbow_upper_limit:=${pi}
+     arm_forearm_lower_limit:=${-pi}    arm_forearm_upper_limit:=${pi}
+     arm_wrist_lower_limit:=${-pi}    arm_wrist_upper_limit:=${pi} -->
+     <!-- arm_elbow_lower_limit:=${-pi}    arm_elbow_upper_limit:=${pi} -->
+     <!-- forearm_lower_limit:=${-pi}    forearm_upper_limit:=${pi} -->
     <!-- Inertia parameters -->
     <xacro:property name="base_mass" value="4.0" />  <!-- This mass might be incorrect -->
@@ -394,6 +402,18 @@
       <child link = "${prefix}fake_hand_link" />
       <origin xyz="0.05 0.0 0.05" rpy="0.0 0.0 0.0" />
-      <!-- <origin xyz="0.0 0.0 0.065" rpy="0.0 0.0 0.0" /> -->
-    </joint>
+    </joint>
+    <!-- <joint name="${prefix}fake_hand_joint" type="revolute">
+      <parent link="${prefix}ee_magnet_cylinder" />
+      <child link = "${prefix}fake_hand_link" />
+      <origin xyz="0.05 0.0 0.05" rpy="0.0 0.0 0.0" />
+      <axis xyz="0 0 1" />
+      <xacro:unless value="${joint_limited}">
+        <limit lower="${-2.0 * pi}" upper="${2.0 * pi}" effort="54.0" velocity="3.2"/>
+      </xacro:unless>
+      <xacro:if value="${joint_limited}">
+        <limit lower="${hand_lower_limit}" upper="${hand_upper_limit}" effort="54.0" velocity="3.2"/>
+      </xacro:if>
+      <dynamics damping="0.0" friction="0.0"/>
+    </joint> -->
     <link name="${prefix}fake_hand_link">
       <visual>
@@ -415,4 +435,159 @@
       </collision>
     </link>
+<!-- #########################ARM TEST########################## -->
+<!-- <joint name="${prefix}fake_forearm_joint" type="fixed">
+  <parent link="${prefix}fake_arm_link" />
+  <child link = "${prefix}fake_forearm_link" />
+  <origin xyz="0.0 0.0 -0.25" rpy="0.0 0.0 0.0" />
+</joint> -->
+<!-- <joint name="${prefix}fake_forearm_joint" type="revolute">
+  <parent link="${prefix}fake_hand_link" />
+  <child link = "${prefix}fake_forearm_link" />
+  <origin xyz="0.0 0.0 -0.25" rpy="0.0 0.0 0.0" />
+  <axis xyz="0 0 1" />
+  <xacro:unless value="${joint_limited}">
+    <limit lower="${-2.0 * pi}" upper="${2.0 * pi}" effort="54.0" velocity="3.2"/>
+  </xacro:unless>
+  <xacro:if value="${joint_limited}">
+    <limit lower="${forearm_lower_limit}" upper="${forearm_upper_limit}" effort="54.0" velocity="3.2"/>
+  </xacro:if>
+  <dynamics damping="0.0" friction="0.0"/>
+</joint>
+    <link name="${prefix}fake_forearm_link">
+      <visual>
+        <geometry>
+          <cylinder length="0.25" radius="0.025"/>
+        </geometry>
+        <origin rpy="0 0 0" xyz="0 0 0"/>
+        <material name="ForearmColor">
+          <color rgba="0.0 0.0 0.0 1.0"/>
+        </material>
+      </visual>
+      <collision>
+        <geometry>
+          <cylinder length="0.25" radius="0.025"/>
+        </geometry>
+        <origin rpy="0 0 0" xyz="0 0 0"/>
+      </collision>
+    </link>
+    <joint name="${prefix}fake_shoulder_joint" type="fixed">
+      <parent link="${prefix}base_link" />
+      <child link = "${prefix}fake_forearm_link" />
+      <origin xyz="0.0 0.0 -0.25" rpy="0.0 0.0 0.0" />
+    </joint> -->
+<!--
+    <link name="${prefix}fake_base_link">
+      <visual>
+        <geometry>
+          <box size="0.1 0.1 0.1"/>
+        </geometry>
+        <origin rpy="0 0 0" xyz="0 0 0"/>
+        <material name="BaseColor">
+          <color rgba="0.0 0.0 1.0 1.0"/>
+        </material>
+      </visual>
+      <collision>
+        <geometry>
+          <box size="0.1 0.1 0.1"/>
+        </geometry>
+        <origin rpy="0 0 0" xyz="0 0 0"/>
+      </collision>
+    </link> -->
+<!-- ################### -->
+    <!-- <joint name="${prefix}arm_shoulder_joint" type="fixed">
+      <parent link="${prefix}base_link" />
+      <child link = "${prefix}arm_shoulder_link" />
+      <origin xyz="-0.15 0.5 0.4" rpy="0.0 0.0 0.0" />
+    </joint>
+    <link name="${prefix}arm_shoulder_link">
+      <visual>
+        <geometry>
+          <box size="0.07 0.07 0.1"/>
+        </geometry>
+        <origin rpy="0 0 0" xyz="0 0 0"/>
+        <material name="ShoulderColour">
+          <color rgba="0.4 0.4 0.4 1.0"/>
+        </material>
+      </visual>
+      <collision>
+        <geometry>
+          <box size="0.05 0.05 0.05"/>
+        </geometry>
+        <origin rpy="0 0 0" xyz="0 0 0"/>
+      </collision>
+    </link>
+    <joint name="${prefix}arm_elbow_joint" type="revolute">
+      <parent link="${prefix}arm_shoulder_link" />
+      <child link = "${prefix}arm_elbow_link" />
+      <origin xyz="0.0 0.0 0.0" rpy="0.0 0.0 0.0" />
+      <axis xyz="0 0 1" />
+      <xacro:unless value="${joint_limited}">
+        <limit lower="${-2.0 * pi}" upper="${2.0 * pi}" effort="54.0" velocity="3.2"/>
+      </xacro:unless>
+      <xacro:if value="${joint_limited}">
+        <limit lower="${arm_elbow_lower_limit}" upper="${arm_elbow_upper_limit}" effort="54.0" velocity="3.2"/>
+      </xacro:if>
+      <dynamics damping="0.0" friction="0.0"/>
+    </joint>
+    <link name="${prefix}arm_elbow_link">
+      <visual>
+        <geometry>
+          <cylinder length="0.3" radius="0.035"/>
+        </geometry>
+        <origin rpy="0 ${pi/2.0} 0" xyz="0.15 0 0"/>
+        <material name="Elbow">
+          <color rgba="0.0 1.0 0.0 1.0"/>
+        </material>
+      </visual>
+      <collision>
+        <geometry>
+          <cylinder length="0.3" radius="0.035"/>
+        </geometry>
+        <origin rpy="0 ${pi/2.0} 0" xyz="0.15 0 0"/>
+      </collision>
+    </link>
+    <joint name="${prefix}arm_forearm_joint" type="revolute">
+      <parent link="${prefix}arm_elbow_link" />
+      <child link = "${prefix}arm_forearm_link" />
+      <origin xyz="0.15 0.0 0.0" rpy="0.0 0.0 0.0" />
+      <axis xyz="0 0 1" />
+      <xacro:unless value="${joint_limited}">
+        <limit lower="${-2.0 * pi}" upper="${2.0 * pi}" effort="54.0" velocity="3.2"/>
+      </xacro:unless>
+      <xacro:if value="${joint_limited}">
+        <limit lower="${arm_forearm_lower_limit}" upper="${arm_forearm_upper_limit}" effort="54.0" velocity="3.2"/>
+      </xacro:if>
+      <dynamics damping="0.0" friction="0.0"/>
+    </joint>
+    <link name="${prefix}arm_forearm_link">
+      <visual>
+        <geometry>
+          <cylinder length="0.25" radius="0.025"/>
+        </geometry>
+        <origin rpy="0 ${pi/2.0} 0" xyz="0.25 0.0 0.0"/>
+        <material name="FA">
+          <color rgba="0.0 0.0 0.0 1.0"/>
+        </material>
+      </visual>
+      <collision>
+        <geometry>
+          <cylinder length="0.25" radius="0.025"/>
+        </geometry>
+        <origin rpy="0 ${pi/2.0} 0" xyz="0.25 0.0 0.0"/>
+      </collision>
+    </link>
+    <joint name="${prefix}arm_wrist_joint" type="revolute">
+      <parent link="${prefix}arm_forearm_link" />
+      <child link = "${prefix}fake_arm_link" />
+      <origin xyz="0.15 0.0 0.0" rpy="0.0 0.0 0.0" />
+      <axis xyz="0 0 1" />
+      <xacro:unless value="${joint_limited}">
+        <limit lower="${-2.0 * pi}" upper="${2.0 * pi}" effort="54.0" velocity="3.2"/>
+      </xacro:unless>
+      <xacro:if value="${joint_limited}">
+        <limit lower="${arm_wrist_lower_limit}" upper="${arm_wrist_upper_limit}" effort="54.0" velocity="3.2"/>
+      </xacro:if>
+      <dynamics damping="0.0" friction="0.0"/>
+    </joint> -->
     <xacro:ur_arm_transmission prefix="${prefix}" />
     <xacro:ur_arm_gazebo prefix="${prefix}" />

File: src/universal_robot/ur_description/urdf/ur10_joint_limited_robot.urdf.xacro (robot description, xacro)
@@ -9,5 +9,5 @@
   <xacro:ur10_robot prefix="" joint_limited="true"
     shoulder_pan_lower_limit="${0}" shoulder_pan_upper_limit="${pi/2}"
-    shoulder_lift_lower_limit="${-4*pi/5}" shoulder_lift_upper_limit="${0}"
+    shoulder_lift_lower_limit="${-pi}" shoulder_lift_upper_limit="${0}"
     elbow_joint_lower_limit="${0}" elbow_joint_upper_limit="${pi}"
     wrist_1_lower_limit="${-pi}" wrist_1_upper_limit="${0}"
@@ -22,2 +22,5 @@
   </joint>
 </robot>
+<!-- arm_elbow_lower_limit="${-pi}" arm_elbow_upper_limit="${pi}"
+arm_forearm_lower_limit="${-pi}" arm_forearm_upper_limit="${pi}"
+arm_wrist_lower_limit="${-pi}" arm_wrist_upper_limit="${pi}" -->

Commit message: Updated robot main urdf. Changed table. Added test service to segmentation. Controller node created (python).

File: src/universal_robot/ur_description/urdf/ur10.urdf.xacro (robot description, xacro)
@@ -292,5 +292,5 @@
       <visual>
         <geometry>
-          <box size="0.085 0.085 0.01"/>
+          <box size="0.09 0.09 0.015"/>
         </geometry>
         <origin rpy="0 ${pi/2.0} 0" xyz="0 0 0"/>
@@ -309,10 +309,10 @@
       <parent link="${prefix}ee_metal_plate" />
       <child link = "${prefix}ee_sensor_plate" />
-      <origin xyz="0.022 0.0 0.0" rpy="0.0 0.0 0.0" />
+      <origin xyz="0.027 0.0 0.0" rpy="0.0 0.0 0.0" />
     </joint>
     <link name="${prefix}ee_sensor_plate">
       <visual>
         <geometry>
-          <cylinder length="0.035" radius="0.06"/>
+          <cylinder length="0.04" radius="0.06"/>
         </geometry>
         <origin rpy="0 ${pi/2.0} 0" xyz="0 0 0"/>
@@ -323,5 +323,5 @@
       <collision>
         <geometry>
-          <cylinder length="0.035" radius="0.06"/>
+          <cylinder length="0.04" radius="0.06"/>
         </geometry>
         <origin rpy="0 ${pi/2.0} 0" xyz="0 0 0"/>
@@ -331,5 +331,5 @@
       <parent link="${prefix}ee_sensor_plate" />
       <child link = "${prefix}ee_magnet_cylinder" />
-      <origin xyz="0.042 0.0 0.0" rpy="0.0 0.0 0.0" />
+      <origin xyz="0.045 0.0 0.0" rpy="0.0 0.0 0.0" />
     </joint>
     <link name="${prefix}ee_magnet_cylinder">
@@ -401,5 +401,5 @@
       <parent link="${prefix}ee_magnet_cylinder" />
       <child link = "${prefix}fake_hand_link" />
-      <origin xyz="0.05 0.0 0.05" rpy="0.0 0.0 0.0" />
+      <origin xyz="0.05 0.0 0.09" rpy="0.0 0.0 0.0" />
     </joint>
     <!-- <joint name="${prefix}fake_hand_joint" type="revolute">
@@ -420,5 +420,5 @@
         <geometry>
           <!-- <box size="0.35 0.05 0.05"/> -->
-          <box size="0.1 0.05 0.05"/>
+          <box size="0.17 0.05 0.05"/>
         </geometry>
         <origin rpy="0 ${pi/2.0} 0" xyz="0 0 0"/>
@@ -430,5 +430,5 @@
         <geometry>
           <!-- <box size="0.35 0.05 0.05"/> -->
-          <box size="0.1 0.05 0.05"/>
+          <box size="0.17 0.05 0.05"/>
         </geometry>
         <origin rpy="0 ${pi/2.0} 0" xyz="0 0 0"/>

File: src/universal_robot/ur_description/urdf/ur10_joint_limited_robot.urdf.xacro (robot description, xacro)
@@ -5,6 +5,6 @@
   <!-- <xacro:include filename="$(find ur_description)/urdf/common.gazebo.xacro" /> -->
   <!-- ur10 -->
-  <!-- <xacro:include filename="$(find ur_description)/urdf/ur10.urdf.xacro" /> -->
-  <xacro:include filename="$(find ur_description)/urdf/Sur10.urdf.xacro" />
+  <xacro:include filename="$(find ur_description)/urdf/ur10.urdf.xacro" />
+  <!-- <xacro:include filename="$(find ur_description)/urdf/Sur10.urdf.xacro" /> -->
   <!-- arm -->
   <xacro:ur10_robot prefix="" joint_limited="true"

Commit message: Before changing controller. Tested IK packages (failed).

File: src/universal_robot/ur_description/urdf/ur10.urdf.xacro (robot description, xacro)
@@ -24,6 +24,6 @@
 		 wrist_3_lower_limit:=${-pi}    wrist_3_upper_limit:=${pi}
      wrist_3_lower_limit:=${-pi}    wrist_3_upper_limit:=${pi}
-     hand_lower_limit:=${-pi}    hand_upper_limit:=${pi}
      ">
+      <!--    hand_lower_limit:=${-pi}    hand_upper_limit:=${pi}-->
      <!-- arm_elbow_lower_limit:=${-pi}    arm_elbow_upper_limit:=${pi}
      arm_forearm_lower_limit:=${-pi}    arm_forearm_upper_limit:=${pi}
@@ -249,5 +249,6 @@
       </xacro:unless>
       <xacro:if value="${joint_limited}">
-        <limit lower="${wrist_3_lower_limit}" upper="${wrist_3_upper_limit}" effort="54.0" velocity="3.2"/>
+      <!--  <limit lower="${wrist_3_lower_limit}" upper="${wrist_3_upper_limit}" effort="54.0" velocity="3.2"/> -->
+        <limit lower="${-pi/2}" upper="${pi/4}" effort="54.0" velocity="3.2"/>
       </xacro:if>
       <dynamics damping="0.0" friction="0.0"/>

File: src/universal_robot/ur_description/urdf/ur10_joint_limited_robot.urdf.xacro (robot description, xacro)
@@ -6,5 +6,5 @@
   <!-- ur10 -->
   <!-- <xacro:include filename="$(find ur_description)/urdf/ur10.urdf.xacro" /> -->
-  <xacro:include filename="$(find ur_description)/urdf/Sur10.urdf.xacro" />
+  <xacro:include filename="$(find ur_description)/urdf/ur10.urdf.xacro" />
   <!-- arm -->
   <xacro:ur10_robot prefix="" joint_limited="true"
@@ -14,5 +14,5 @@
     wrist_1_lower_limit="${-pi}" wrist_1_upper_limit="${0}"
     wrist_2_lower_limit="${-pi}" wrist_2_upper_limit="${pi/4}"
-    wrist_3_lower_limit="${-pi}" wrist_3_upper_limit="${pi}"
+    wrist_3_lower_limit="${-pi/2}" wrist_3_upper_limit="${0}"
 />
   <link name="world" />

Commit message: Fixed gase optimiser service + interaction with controller node. Changed hand URDF (thinner). Added getpositionFK service (not working)

File: src/universal_robot/ur_description/urdf/ur10.urdf.xacro (robot description, xacro)
@@ -421,5 +421,5 @@
         <geometry>
           <!-- <box size="0.35 0.05 0.05"/> -->
-          <box size="0.17 0.05 0.05"/>
+          <box size="0.17 0.03 0.05"/>
         </geometry>
         <origin rpy="0 ${pi/2.0} 0" xyz="0 0 0"/>
@@ -431,5 +431,5 @@
         <geometry>
           <!-- <box size="0.35 0.05 0.05"/> -->
-          <box size="0.17 0.05 0.05"/>
+          <box size="0.17 0.03 0.05"/>
         </geometry>
         <origin rpy="0 ${pi/2.0} 0" xyz="0 0 0"/>

Commit message: Implemented IK model. Plot 2D objects, plot arm

File: src/universal_robot/ur_description/urdf/ur10.urdf.xacro (robot description, xacro)
@@ -249,6 +249,6 @@
       </xacro:unless>
       <xacro:if value="${joint_limited}">
-      <!--  <limit lower="${wrist_3_lower_limit}" upper="${wrist_3_upper_limit}" effort="54.0" velocity="3.2"/> -->
-        <limit lower="${-pi/2}" upper="${pi/4}" effort="54.0" velocity="3.2"/>
+       <limit lower="${wrist_3_lower_limit}" upper="${wrist_3_upper_limit}" effort="54.0" velocity="3.2"/>
+        <!-- <limit lower="${-pi/2}" upper="${pi/4}" effort="54.0" velocity="3.2"/> -->
       </xacro:if>
       <dynamics damping="0.0" friction="0.0"/>

File: src/universal_robot/ur_description/urdf/ur10_joint_limited_robot.urdf.xacro (robot description, xacro)
@@ -14,5 +14,5 @@
     wrist_1_lower_limit="${-pi}" wrist_1_upper_limit="${0}"
     wrist_2_lower_limit="${-pi}" wrist_2_upper_limit="${pi/4}"
-    wrist_3_lower_limit="${-pi/2}" wrist_3_upper_limit="${0}"
+    wrist_3_lower_limit="${-pi}" wrist_3_upper_limit="${pi}"
 />
   <link name="world" />

Commit message: Changed UDRF fake_hand_link. Fixed IK calculations.

File: src/universal_robot/ur_description/urdf/ur10.urdf.xacro (robot description, xacro)
@@ -377,5 +377,5 @@
       </collision>
     </link> -->
-    <joint name="${prefix}fake_arm_joint" type="fixed">
+    <!-- <joint name="${prefix}fake_arm_joint" type="fixed">
       <parent link="${prefix}ee_magnet_cylinder" />
       <child link = "${prefix}fake_arm_link" />
@@ -398,9 +398,9 @@
         <origin rpy="0 0 0" xyz="0 0 0"/>
       </collision>
-    </link>
+    </link> -->
     <joint name="${prefix}fake_hand_joint" type="fixed">
       <parent link="${prefix}ee_magnet_cylinder" />
       <child link = "${prefix}fake_hand_link" />
-      <origin xyz="0.05 0.0 0.09" rpy="0.0 0.0 0.0" />
+      <origin xyz="0.05 0.0 0.025" rpy="0.0 0.0 0.0" />
     </joint>
     <!-- <joint name="${prefix}fake_hand_joint" type="revolute">
@@ -421,5 +421,5 @@
         <geometry>
           <!-- <box size="0.35 0.05 0.05"/> -->
-          <box size="0.17 0.03 0.05"/>
+          <box size="0.13 0.03 0.05"/>
         </geometry>
         <origin rpy="0 ${pi/2.0} 0" xyz="0 0 0"/>
@@ -431,5 +431,5 @@
         <geometry>
           <!-- <box size="0.35 0.05 0.05"/> -->
-          <box size="0.17 0.03 0.05"/>
+          <box size="0.13 0.03 0.05"/>
         </geometry>
         <origin rpy="0 ${pi/2.0} 0" xyz="0 0 0"/>

Commit message: Changed URDf fake hand link

File: src/universal_robot/ur_description/urdf/ur10.urdf.xacro (robot description, xacro)
@@ -399,8 +399,8 @@
       </collision>
     </link> -->
-    <joint name="${prefix}fake_hand_joint" type="fixed">
+    <joint name="${prefix}fake_wrist_joint" type="fixed">
       <parent link="${prefix}ee_magnet_cylinder" />
-      <child link = "${prefix}fake_hand_link" />
-      <origin xyz="0.05 0.0 0.025" rpy="0.0 0.0 0.0" />
+      <child link = "${prefix}fake_wrist_link" />
+      <origin xyz="0.05 0.0 0.0" rpy="0.0 0.0 0.0" />
     </joint>
     <!-- <joint name="${prefix}fake_hand_joint" type="revolute">
@@ -417,13 +417,37 @@
       <dynamics damping="0.0" friction="0.0"/>
     </joint> -->
+    <link name="${prefix}fake_wrist_link">
+      <visual>
+        <geometry>
+          <!-- <box size="0.35 0.05 0.05"/> -->
+          <box size="0.08 0.03 0.05"/>
+        </geometry>
+        <origin rpy="0 ${pi/2.0} 0" xyz="0 0 0"/>
+        <material name="WristColor">
+          <color rgba="0.4 0.4 0.4 1.0"/>
+        </material>
+      </visual>
+      <collision>
+        <geometry>
+          <!-- <box size="0.35 0.05 0.05"/> -->
+          <box size="0.08 0.03 0.05"/>
+        </geometry>
+        <origin rpy="0 ${pi/2.0} 0" xyz="0 0 0"/>
+      </collision>
+    </link>
+    <joint name="${prefix}fake_hand_joint" type="fixed">
+      <parent link="${prefix}fake_wrist_link" />
+      <child link = "${prefix}fake_hand_link" />
+      <origin xyz="0.0 0.0 0.09" rpy="0.0 0.0 0.0" />
+    </joint>
     <link name="${prefix}fake_hand_link">
       <visual>
         <geometry>
           <!-- <box size="0.35 0.05 0.05"/> -->
-          <box size="0.13 0.03 0.05"/>
-        </geometry>
-        <origin rpy="0 ${pi/2.0} 0" xyz="0 0 0"/>
-        <material name="HandColor">
-          <color rgba="0.4 0.4 0.4 1.0"/>
+          <box size="0.10 0.03 0.05"/>
+        </geometry>
+        <origin rpy="0 ${pi/2.0} 0" xyz="0 0 0"/>
+        <material name="handColor">
+          <color rgba="0.2 0.2 0.2 1.0"/>
         </material>
       </visual>
@@ -431,5 +455,5 @@
         <geometry>
           <!-- <box size="0.35 0.05 0.05"/> -->
-          <box size="0.13 0.03 0.05"/>
+          <box size="0.10 0.03 0.05"/>
         </geometry>
         <origin rpy="0 ${pi/2.0} 0" xyz="0 0 0"/>

Commit message: First attempt of orientation control

File: src/universal_robot/ur_description/urdf/ur10.urdf.xacro (robot description, xacro)
@@ -446,4 +446,5 @@
           <!-- <box size="0.35 0.05 0.05"/> -->
           <box size="0.10 0.03 0.05"/>
+          <!--<mesh filename="package://ur_description/meshes/hand.stl"/>-->
         </geometry>
         <origin rpy="0 ${pi/2.0} 0" xyz="0 0 0"/>
@@ -456,4 +457,5 @@
           <!-- <box size="0.35 0.05 0.05"/> -->
           <box size="0.10 0.03 0.05"/>
+          <!--<mesh filename="package://ur_description/meshes/hand.stl"/>-->
         </geometry>
         <origin rpy="0 ${pi/2.0} 0" xyz="0 0 0"/>
