Commit message: Tested with robot, fix offsets

File: src/universal_robot/ur_description/urdf/ur10.urdf.xacro (robot description, xacro)
@@ -439,5 +439,5 @@
       <parent link="${prefix}fake_wrist_link" />
       <child link = "${prefix}fake_hand_link" />
-      <origin xyz="0.0 0.0 0.09" rpy="0.0 0.0 0.0" />
+      <origin xyz="0.0 0.0 0.10" rpy="0.0 0.0 0.0" />
     </joint>
     <link name="${prefix}fake_hand_link">
@@ -445,5 +445,5 @@
         <geometry>
           <!-- <box size="0.35 0.05 0.05"/> -->
-          <box size="0.10 0.03 0.05"/>
+          <box size="0.15 0.03 0.05"/>
           <!--<mesh filename="package://ur_description/meshes/hand.stl"/>-->
         </geometry>
@@ -456,5 +456,5 @@
         <geometry>
           <!-- <box size="0.35 0.05 0.05"/> -->
-          <box size="0.10 0.03 0.05"/>
+          <box size="0.15 0.03 0.05"/>
           <!--<mesh filename="package://ur_description/meshes/hand.stl"/>-->
         </geometry>

Commit message: Added points to table of pointcloud - test more

File: src/universal_robot/ur_description/urdf/ur10.urdf.xacro (robot description, xacro)
@@ -439,5 +439,5 @@
       <parent link="${prefix}fake_wrist_link" />
       <child link = "${prefix}fake_hand_link" />
-      <origin xyz="0.0 0.0 0.10" rpy="0.0 0.0 0.0" />
+      <origin xyz="0.0 0.0 0.115" rpy="0.0 0.0 0.0" />
     </joint>
     <link name="${prefix}fake_hand_link">

Commit message: Corrected URDF, changed grasp point

File: src/universal_robot/ur_description/urdf/ur10.urdf.xacro (robot description, xacro)
@@ -439,5 +439,5 @@
       <parent link="${prefix}fake_wrist_link" />
       <child link = "${prefix}fake_hand_link" />
-      <origin xyz="0.0 0.0 0.115" rpy="0.0 0.0 0.0" />
+      <origin xyz="0.0 0.0 0.095" rpy="0.0 0.0 0.0" />  #0.115 offsey for 0.15 hand length
     </joint>
     <link name="${prefix}fake_hand_link">
@@ -445,5 +445,5 @@
         <geometry>
           <!-- <box size="0.35 0.05 0.05"/> -->
-          <box size="0.15 0.03 0.05"/>
+          <box size="0.11 0.03 0.05"/>
           <!--<mesh filename="package://ur_description/meshes/hand.stl"/>-->
         </geometry>
@@ -456,5 +456,5 @@
         <geometry>
           <!-- <box size="0.35 0.05 0.05"/> -->
-          <box size="0.15 0.03 0.05"/>
+          <box size="0.11 0.03 0.05"/>
           <!--<mesh filename="package://ur_description/meshes/hand.stl"/>-->
         </geometry>

Commit message: Fixed mapping memory issues

File: src/universal_robot/ur_description/urdf/ur10.urdf.xacro (robot description, xacro)
@@ -439,5 +439,5 @@
       <parent link="${prefix}fake_wrist_link" />
       <child link = "${prefix}fake_hand_link" />
-      <origin xyz="0.0 0.0 0.095" rpy="0.0 0.0 0.0" />  #0.115 offsey for 0.15 hand length
+      <origin xyz="0.0 0.0 0.095" rpy="0.0 0.0 0.0" />  #0.115 offset for 0.15 hand length
     </joint>
     <link name="${prefix}fake_hand_link">

Commit message: After 2 participant

File: src/universal_robot/ur_description/urdf/ur10.urdf.xacro (robot description, xacro)
@@ -402,5 +402,5 @@
       <parent link="${prefix}ee_magnet_cylinder" />
       <child link = "${prefix}fake_wrist_link" />
-      <origin xyz="0.05 0.0 0.0" rpy="0.0 0.0 0.0" />
+      <origin xyz="0.07 0.0 0.0" rpy="0.0 0.0 0.0" />
     </joint>
     <!-- <joint name="${prefix}fake_hand_joint" type="revolute">
@@ -421,5 +421,5 @@
         <geometry>
           <!-- <box size="0.35 0.05 0.05"/> -->
-          <box size="0.08 0.03 0.05"/>
+          <box size="0.08 0.04 0.09"/>
         </geometry>
         <origin rpy="0 ${pi/2.0} 0" xyz="0 0 0"/>
@@ -431,5 +431,5 @@
         <geometry>
           <!-- <box size="0.35 0.05 0.05"/> -->
-          <box size="0.08 0.03 0.05"/>
+          <box size="0.08 0.03 0.09"/>
         </geometry>
         <origin rpy="0 ${pi/2.0} 0" xyz="0 0 0"/>
@@ -445,5 +445,5 @@
         <geometry>
           <!-- <box size="0.35 0.05 0.05"/> -->
-          <box size="0.11 0.03 0.05"/>
+          <box size="0.11 0.04 0.05"/>
           <!--<mesh filename="package://ur_description/meshes/hand.stl"/>-->
         </geometry>
@@ -456,5 +456,5 @@
         <geometry>
           <!-- <box size="0.35 0.05 0.05"/> -->
-          <box size="0.11 0.03 0.05"/>
+          <box size="0.11 0.04 0.05"/>
           <!--<mesh filename="package://ur_description/meshes/hand.stl"/>-->
         </geometry>

Commit message: All code cleaned and commented

File: src/universal_robot/ur_description/urdf/ur10.urdf.xacro (robot description, xacro)
@@ -25,10 +25,4 @@
      wrist_3_lower_limit:=${-pi}    wrist_3_upper_limit:=${pi}
      ">
-      <!--    hand_lower_limit:=${-pi}    hand_upper_limit:=${pi}-->
-     <!-- arm_elbow_lower_limit:=${-pi}    arm_elbow_upper_limit:=${pi}
-     arm_forearm_lower_limit:=${-pi}    arm_forearm_upper_limit:=${pi}
-     arm_wrist_lower_limit:=${-pi}    arm_wrist_upper_limit:=${pi} -->
-     <!-- arm_elbow_lower_limit:=${-pi}    arm_elbow_upper_limit:=${pi} -->
-     <!-- forearm_lower_limit:=${-pi}    forearm_upper_limit:=${pi} -->
     <!-- Inertia parameters -->
     <xacro:property name="base_mass" value="4.0" />  <!-- This mass might be incorrect -->
@@ -285,4 +279,6 @@
       </collision>
     </link>
+    <!-- The next links and joints were added to the standard Ur10 URDF -->
+    <!-- Joint and link for the metal plate connected to the ee link -->
     <joint name="${prefix}ee_plate_joint" type="fixed">
       <parent link="${prefix}ee_link" />
@@ -307,4 +303,5 @@
       </collision>
     </link>
+    <!-- Joint and link for the force sensor -->
     <joint name="${prefix}ee_sensor_joint" type="fixed">
       <parent link="${prefix}ee_metal_plate" />
@@ -329,4 +326,5 @@
       </collision>
     </link>
+    <!-- Joint and link for the magnetic attachment connected to the force sensor -->
     <joint name="${prefix}ee_magnet_joint" type="fixed">
       <parent link="${prefix}ee_sensor_plate" />
@@ -351,52 +349,5 @@
       </collision>
     </link>
-<!--
-    <joint name="${prefix}fake_hand_joint" type="fixed">
-      <parent link="${prefix}ee_magnet_cylinder" />
-      <child link = "${prefix}fake_hand_link" />
-      <origin xyz="0.05 0.0 -0.05" rpy="0.0 0.0 0.0" /> -->
-      <!-- <origin xyz="0.0 0.0 0.065" rpy="0.0 0.0 0.0" /> -->
-    <!-- </joint> -->
-    <!-- <link name="${prefix}fake_hand_link">
-      <visual>
-        <geometry>
-          <box size="0.35 0.05 0.05"/> -->
-          <!-- <box size="0.08 0.05 0.05"/> -->
-        <!-- </geometry>
-        <origin rpy="0 ${pi/2.0} 0" xyz="0 0 0"/>
-        <material name="HandColor">
-          <color rgba="0.4 0.4 0.4 1.0"/>
-        </material>
-      </visual>
-      <collision>
-        <geometry>
-          <box size="0.35 0.05 0.05"/> -->
-          <!-- <box size="0.08 0.05 0.05"/> -->
-        <!-- </geometry>
-        <origin rpy="0 ${pi/2.0} 0" xyz="0 0 0"/>
-      </collision>
-    </link> -->
-    <!-- <joint name="${prefix}fake_arm_joint" type="fixed">
-      <parent link="${prefix}ee_magnet_cylinder" />
-      <child link = "${prefix}fake_arm_link" />
-      <origin xyz="0.05 0.0 -0.12" rpy="0.0 0.0 0.0" />
-    </joint>
-    <link name="${prefix}fake_arm_link">
-      <visual>
-        <geometry>
-          <cylinder length="0.25" radius="0.025"/>
-        </geometry>
-        <origin rpy="0 0 0" xyz="0 0 0"/>
-        <material name="ArmColor">
-          <color rgba="1.0 1.0 1.0 1.0"/>
-        </material>
-      </visual>
-      <collision>
-        <geometry>
-          <cylinder length="0.25" radius="0.025"/>
-        </geometry>
-        <origin rpy="0 0 0" xyz="0 0 0"/>
-      </collision>
-    </link> -->
+    <!-- Joint and link that represent the human wrist -->
     <joint name="${prefix}fake_wrist_joint" type="fixed">
       <parent link="${prefix}ee_magnet_cylinder" />
@@ -404,21 +355,7 @@
       <origin xyz="0.07 0.0 0.0" rpy="0.0 0.0 0.0" />
     </joint>
-    <!-- <joint name="${prefix}fake_hand_joint" type="revolute">
-      <parent link="${prefix}ee_magnet_cylinder" />
-      <child link = "${prefix}fake_hand_link" />
-      <origin xyz="0.05 0.0 0.05" rpy="0.0 0.0 0.0" />
-      <axis xyz="0 0 1" />
-      <xacro:unless value="${joint_limited}">
-        <limit lower="${-2.0 * pi}" upper="${2.0 * pi}" effort="54.0" velocity="3.2"/>
-      </xacro:unless>
-      <xacro:if value="${joint_limited}">
-        <limit lower="${hand_lower_limit}" upper="${hand_upper_limit}" effort="54.0" velocity="3.2"/>
-      </xacro:if>
-      <dynamics damping="0.0" friction="0.0"/>
-    </joint> -->
     <link name="${prefix}fake_wrist_link">
       <visual>
         <geometry>
-          <!-- <box size="0.35 0.05 0.05"/> -->
           <box size="0.08 0.04 0.09"/>
         </geometry>
@@ -430,5 +367,4 @@
       <collision>
         <geometry>
-          <!-- <box size="0.35 0.05 0.05"/> -->
           <box size="0.08 0.03 0.09"/>
         </geometry>
@@ -436,4 +372,5 @@
       </collision>
     </link>
+    <!-- Joint and link that represent the human hand -->
     <joint name="${prefix}fake_hand_joint" type="fixed">
       <parent link="${prefix}fake_wrist_link" />
@@ -444,7 +381,5 @@
       <visual>
         <geometry>
-          <!-- <box size="0.35 0.05 0.05"/> -->
           <box size="0.11 0.04 0.05"/>
-          <!--<mesh filename="package://ur_description/meshes/hand.stl"/>-->
         </geometry>
         <origin rpy="0 ${pi/2.0} 0" xyz="0 0 0"/>
@@ -455,166 +390,9 @@
       <collision>
         <geometry>
-          <!-- <box size="0.35 0.05 0.05"/> -->
           <box size="0.11 0.04 0.05"/>
-          <!--<mesh filename="package://ur_description/meshes/hand.stl"/>-->
-        </geometry>
-        <origin rpy="0 ${pi/2.0} 0" xyz="0 0 0"/>
-      </collision>
-    </link>
-<!-- #########################ARM TEST########################## -->
-<!-- <joint name="${prefix}fake_forearm_joint" type="fixed">
-  <parent link="${prefix}fake_arm_link" />
-  <child link = "${prefix}fake_forearm_link" />
-  <origin xyz="0.0 0.0 -0.25" rpy="0.0 0.0 0.0" />
-</joint> -->
-<!-- <joint name="${prefix}fake_forearm_joint" type="revolute">
-  <parent link="${prefix}fake_hand_link" />
-  <child link = "${prefix}fake_forearm_link" />
-  <origin xyz="0.0 0.0 -0.25" rpy="0.0 0.0 0.0" />
-  <axis xyz="0 0 1" />
-  <xacro:unless value="${joint_limited}">
-    <limit lower="${-2.0 * pi}" upper="${2.0 * pi}" effort="54.0" velocity="3.2"/>
-  </xacro:unless>
-  <xacro:if value="${joint_limited}">
-    <limit lower="${forearm_lower_limit}" upper="${forearm_upper_limit}" effort="54.0" velocity="3.2"/>
-  </xacro:if>
-  <dynamics damping="0.0" friction="0.0"/>
-</joint>
-    <link name="${prefix}fake_forearm_link">
-      <visual>
-        <geometry>
-          <cylinder length="0.25" radius="0.025"/>
-        </geometry>
-        <origin rpy="0 0 0" xyz="0 0 0"/>
-        <material name="ForearmColor">
-          <color rgba="0.0 0.0 0.0 1.0"/>
-        </material>
-      </visual>
-      <collision>
-        <geometry>
-          <cylinder length="0.25" radius="0.025"/>
-        </geometry>
-        <origin rpy="0 0 0" xyz="0 0 0"/>
-      </collision>
-    </link>
-    <joint name="${prefix}fake_shoulder_joint" type="fixed">
-      <parent link="${prefix}base_link" />
-      <child link = "${prefix}fake_forearm_link" />
-      <origin xyz="0.0 0.0 -0.25" rpy="0.0 0.0 0.0" />
-    </joint> -->
-<!--
-    <link name="${prefix}fake_base_link">
-      <visual>
-        <geometry>
-          <box size="0.1 0.1 0.1"/>
-        </geometry>
-        <origin rpy="0 0 0" xyz="0 0 0"/>
-        <material name="BaseColor">
-          <color rgba="0.0 0.0 1.0 1.0"/>
-        </material>
-      </visual>
-      <collision>
-        <geometry>
-          <box size="0.1 0.1 0.1"/>
-        </geometry>
-        <origin rpy="0 0 0" xyz="0 0 0"/>
-      </collision>
-    </link> -->
-<!-- ################### -->
-    <!-- <joint name="${prefix}arm_shoulder_joint" type="fixed">
-      <parent link="${prefix}base_link" />
-      <child link = "${prefix}arm_shoulder_link" />
-      <origin xyz="-0.15 0.5 0.4" rpy="0.0 0.0 0.0" />
-    </joint>
-    <link name="${prefix}arm_shoulder_link">
-      <visual>
-        <geometry>
-          <box size="0.07 0.07 0.1"/>
-        </geometry>
-        <origin rpy="0 0 0" xyz="0 0 0"/>
-        <material name="ShoulderColour">
-          <color rgba="0.4 0.4 0.4 1.0"/>
-        </material>
-      </visual>
-      <collision>
-        <geometry>
-          <box size="0.05 0.05 0.05"/>
-        </geometry>
-        <origin rpy="0 0 0" xyz="0 0 0"/>
-      </collision>
-    </link>
-    <joint name="${prefix}arm_elbow_joint" type="revolute">
-      <parent link="${prefix}arm_shoulder_link" />
-      <child link = "${prefix}arm_elbow_link" />
-      <origin xyz="0.0 0.0 0.0" rpy="0.0 0.0 0.0" />
-      <axis xyz="0 0 1" />
-      <xacro:unless value="${joint_limited}">
-        <limit lower="${-2.0 * pi}" upper="${2.0 * pi}" effort="54.0" velocity="3.2"/>
-      </xacro:unless>
-      <xacro:if value="${joint_limited}">
-        <limit lower="${arm_elbow_lower_limit}" upper="${arm_elbow_upper_limit}" effort="54.0" velocity="3.2"/>
-      </xacro:if>
-      <dynamics damping="0.0" friction="0.0"/>
-    </joint>
-    <link name="${prefix}arm_elbow_link">
-      <visual>
-        <geometry>
-          <cylinder length="0.3" radius="0.035"/>
-        </geometry>
-        <origin rpy="0 ${pi/2.0} 0" xyz="0.15 0 0"/>
-        <material name="Elbow">
-          <color rgba="0.0 1.0 0.0 1.0"/>
-        </material>
-      </visual>
-      <collision>
-        <geometry>
-          <cylinder length="0.3" radius="0.035"/>
-        </geometry>
-        <origin rpy="0 ${pi/2.0} 0" xyz="0.15 0 0"/>
-      </collision>
-    </link>
-    <joint name="${prefix}arm_forearm_joint" type="revolute">
-      <parent link="${prefix}arm_elbow_link" />
-      <child link = "${prefix}arm_forearm_link" />
-      <origin xyz="0.15 0.0 0.0" rpy="0.0 0.0 0.0" />
-      <axis xyz="0 0 1" />
-      <xacro:unless value="${joint_limited}">
-        <limit lower="${-2.0 * pi}" upper="${2.0 * pi}" effort="54.0" velocity="3.2"/>
-      </xacro:unless>
-      <xacro:if value="${joint_limited}">
-        <limit lower="${arm_forearm_lower_limit}" upper="${arm_forearm_upper_limit}" effort="54.0" velocity="3.2"/>
-      </xacro:if>
-      <dynamics damping="0.0" friction="0.0"/>
-    </joint>
-    <link name="${prefix}arm_forearm_link">
-      <visual>
-        <geometry>
-          <cylinder length="0.25" radius="0.025"/>
-        </geometry>
-        <origin rpy="0 ${pi/2.0} 0" xyz="0.25 0.0 0.0"/>
-        <material name="FA">
-          <color rgba="0.0 0.0 0.0 1.0"/>
-        </material>
-      </visual>
-      <collision>
-        <geometry>
-          <cylinder length="0.25" radius="0.025"/>
-        </geometry>
-        <origin rpy="0 ${pi/2.0} 0" xyz="0.25 0.0 0.0"/>
-      </collision>
-    </link>
-    <joint name="${prefix}arm_wrist_joint" type="revolute">
-      <parent link="${prefix}arm_forearm_link" />
-      <child link = "${prefix}fake_arm_link" />
-      <origin xyz="0.15 0.0 0.0" rpy="0.0 0.0 0.0" />
-      <axis xyz="0 0 1" />
-      <xacro:unless value="${joint_limited}">
-        <limit lower="${-2.0 * pi}" upper="${2.0 * pi}" effort="54.0" velocity="3.2"/>
-      </xacro:unless>
-      <xacro:if value="${joint_limited}">
-        <limit lower="${arm_wrist_lower_limit}" upper="${arm_wrist_upper_limit}" effort="54.0" velocity="3.2"/>
-      </xacro:if>
-      <dynamics damping="0.0" friction="0.0"/>
-    </joint> -->
+        </geometry>
+        <origin rpy="0 ${pi/2.0} 0" xyz="0 0 0"/>
+      </collision>
+    </link>
     <xacro:ur_arm_transmission prefix="${prefix}" />
     <xacro:ur_arm_gazebo prefix="${prefix}" />
